Commit message: Fix formatting in xacro file.

File: urdf/link_calibration.urdf.xacro (robot description, xacro)
@@ -5,10 +5,9 @@
     <link name="${name}">
       <inertial>
-        <origin xyz="0 0 1" rpy="0 0 0"/>
-        <mass value="0.01"/>
-        <inertia
-          ixx="1.0" ixy="0.0" ixz="0.0"
-          iyy="1.0" iyz="0.0"
-          izz="1.0"/>
+        <origin xyz="0 0 1" rpy="0 0 0" />
+        <mass value="0.01" />
+        <inertia ixx="1.0" ixy="0.0" ixz="0.0"
+                 iyy="1.0" iyz="0.0"
+                 izz="1.0" />
       </inertial>
     </link>
@@ -19,6 +18,6 @@
       <parent link="${parent}" />
       <child link="${name}" />
-      <axis xyz="${axis}"/>
-      <limit lower="-0.5" upper="+0.5" effort="999" velocity="999"/>
+      <axis xyz="${axis}" />
+      <limit lower="-0.5" upper="+0.5" effort="999" velocity="999" />
     </joint>
   </xacro:macro>
@@ -28,6 +27,6 @@
       <parent link="${parent}" />
       <child link="${name}" />
-      <axis xyz="${axis}"/>
-      <limit lower="-0.5" upper="+0.5" effort="999" velocity="999"/>
+      <axis xyz="${axis}" />
+      <limit lower="-0.5" upper="+0.5" effort="999" velocity="999" />
     </joint>
   </xacro:macro>
@@ -49,6 +48,6 @@
     <!-- Base offset -->
     <joint name="${name}_joint" type="fixed">
-      <parent link="${parent}"/>
-      <child link="${name}_base"/>
+      <parent link="${parent}" />
+      <child link="${name}_base" />
       <origin xyz="${translateX} ${translateY} ${translateZ}" rpy="${rotX} ${rotY} ${rotZ}" />
     </joint>
@@ -58,20 +57,20 @@
     <prismatic_calibration_joint name="${name}_y_offset"
                                  parent="${name}_x_offset"
-                                 axis="0 1 0"/>
+                                 axis="0 1 0" />
     <prismatic_calibration_joint name="${name}_z_offset"
                                  parent="${name}_y_offset"
-                                 axis="0 0 1"/>
+                                 axis="0 0 1" />
     <revolute_calibration_joint name="${name}_pitch"
                                 parent="${name}_z_offset"
-                                axis="0 1 0"/>
+                                axis="0 1 0" />
     <revolute_calibration_joint name="${name}_roll"
                                 parent="${name}_pitch"
-                                axis="1 0 0"/>
+                                axis="1 0 0" />
     <revolute_calibration_joint name="${name}_yaw"
                                 parent="${name}_roll"
-                                axis="0 0 1"/>
+                                axis="0 0 1" />
     <joint name="${name}_final_joint" type="fixed">
-      <parent link="${name}_yaw"/>
-      <child link="${name}"/>
+      <parent link="${name}_yaw" />
+      <child link="${name}" />
     </joint>
   </xacro:macro>
