Commit message: Fix incorrect measurement.

File: urdf/automower_ipw.urdf.xacro (robot description, xacro)
@@ -4,5 +4,5 @@
   <xacro:include filename="$(find oru_ipw_description)/urdf/link_calibration.urdf.xacro" />
   <!-- Various measurements -->
-  <xacro:property name="frame_xoff_base_link" value="-0.134" />
+  <xacro:property name="frame_xoff_base_link" value="-0.10" />
   <xacro:property name="frame_zoff_base_link" value="0.18041" />
   <xacro:property name="realsense_xoff_frame" value="0.46" />

Commit message: Add reversed base link frame as an experiment.

File: urdf/automower_ipw.urdf.xacro (robot description, xacro)
@@ -2,5 +2,5 @@
 <robot name="automower_ipw" xmlns:xacro="http://www.ros.org/wiki/xacro">
   <xacro:include filename="$(find am_description)/urdf/automower.urdf.xacro" />
-  <xacro:include filename="$(find oru_ipw_description)/urdf/link_calibration.urdf.xacro" />
+  <xacro:include filename="$(find oru_ipw_description)/urdf/links.urdf.xacro" />
   <!-- Various measurements -->
   <xacro:property name="frame_xoff_base_link" value="-0.10" />
@@ -11,4 +11,5 @@
   <!-- From Velodyne datasheet -->
   <xacro:property name="velodyne_laser_center_zoff" value="0.0378" />
+  <fixed_link name="base_link_inverted" parent="base_link" rotZ="${M_PI}" />
   <!-- Define some helper TF frames -->
   <!-- Middle of back aluminum profile, on the upper inside (marked with black pen) -->

File: urdf/links.urdf.xacro (robot description, xacro)
@@ -29,4 +29,19 @@
       <axis xyz="${axis}" />
       <limit lower="-0.5" upper="+0.5" effort="999" velocity="999" />
+    </joint>
+  </xacro:macro>
+  <!-- NOTE! Must have a mass/inertial so that Gazebo does not ignore these... -->
+  <xacro:macro name="fixed_link"
+               params="name parent translateX:=0 translateY:=0 translateZ:=0 rotX:=0.0 rotY:=0.0 rotZ:=0.0">
+    <inertial_link name="${name}" />
+    <gazebo reference="${name}">
+      <turnGravityOff>true</turnGravityOff>
+      <material>Gazebo/Orange</material>
+    </gazebo>
+    <!-- Base offset -->
+    <joint name="${name}_joint" type="fixed">
+      <parent link="${parent}" />
+      <child link="${name}" />
+      <origin xyz="${translateX} ${translateY} ${translateZ}" rpy="${rotX} ${rotY} ${rotZ}" />
     </joint>
   </xacro:macro>

Commit message: Create base_footprint link as parent of base_link

File: urdf/automower_ipw.urdf.xacro (robot description, xacro)
@@ -4,4 +4,5 @@
   <xacro:include filename="$(find oru_ipw_description)/urdf/links.urdf.xacro" />
   <!-- Various measurements -->
+  <xacro:property name="base_link_zoff_base_footprint" value="0.1225" />
   <xacro:property name="frame_xoff_base_link" value="-0.10" />
   <xacro:property name="frame_zoff_base_link" value="0.18041" />
@@ -11,4 +12,15 @@
   <!-- From Velodyne datasheet -->
   <xacro:property name="velodyne_laser_center_zoff" value="0.0378" />
+  <!-- Add base_footprint TF entry -->
+  <link name="base_footprint" />
+  <gazebo reference="base_footprint">
+    <turnGravityOff>true</turnGravityOff>
+    <material>Gazebo/Orange</material>
+  </gazebo>
+  <joint name="base_footprint_joint" type="fixed">
+    <parent link="base_footprint" />
+    <child link="base_link" />
+    <origin xyz="0 0 ${base_link_zoff_base_footprint}" rpy="0 0 0" />
+  </joint>
   <fixed_link name="base_link_inverted" parent="base_link" rotZ="${M_PI}" />
   <!-- Define some helper TF frames -->

Commit message: Lower the laser physically and thus adjust the URDF.

File: urdf/automower_ipw.urdf.xacro (robot description, xacro)
@@ -8,6 +8,8 @@
   <xacro:property name="frame_zoff_base_link" value="0.18041" />
   <xacro:property name="realsense_xoff_frame" value="0.46" />
+  <xacro:property name="realsense_zoff_frame" value="0.06" />
+  <xacro:property name="velodyne_base_zoff_frame" value="0.326" />
   <xacro:property name="velodyne_xoff_frame" value="${0.245 + 0.02 + 0.0774}" />
-  <xacro:property name="velodyne_base_zoff_frame" value="0.41" />
+  <xacro:property name="velodyne_base_thickness" value="0.01" />
   <!-- From Velodyne datasheet -->
   <xacro:property name="velodyne_laser_center_zoff" value="0.0378" />
@@ -29,16 +31,16 @@
                     parent="base_link"
                     translateX="${frame_xoff_base_link}"
-                    translateY="0.0"
                     translateZ="${frame_zoff_base_link}" />
+  <fixed_link name="velodyne_beam_link"
+              parent="mounting_frame_link"
+              translateX="${velodyne_xoff_frame}"
+              translateZ="${velodyne_base_zoff_frame}" />
   <!-- Define extra sensors -->
   <link_calibration name="velodyne"
-                    parent="mounting_frame_link"
-                    translateX="${velodyne_xoff_frame}"
-                    translateY="0.0"
-                    translateZ="${velodyne_base_zoff_frame + velodyne_laser_center_zoff}" />
+                    parent="velodyne_beam_link"
+                    translateZ="${velodyne_base_thickness + velodyne_laser_center_zoff}" />
   <link_calibration name="camera_link"
                     parent="mounting_frame_link"
                     translateX="${realsense_xoff_frame}"
-                    translateY="0.0"
-                    translateZ="0.0" />
+                    translateZ="${realsense_zoff_frame}" />
 </robot>

File: urdf/links.urdf.xacro (robot description, xacro)
@@ -48,5 +48,5 @@
   <!-- NOTE! Must have a mass/inertial so that Gazebo does not ignore these... -->
   <xacro:macro name="link_calibration"
-               params="name parent translateX translateY translateZ rotX:=0.0 rotY:=0.0 rotZ:=0.0">
+               params="name parent translateX:=0.0 translateY:=0.0 translateZ:=0.0 rotX:=0.0 rotY:=0.0 rotZ:=0.0">
     <inertial_link name="${name}_base" />
     <inertial_link name="${name}_x_offset" />

Commit message: Switch camera

File: urdf/automower_ipw.urdf.xacro (robot description, xacro)
@@ -7,6 +7,6 @@
   <xacro:property name="frame_xoff_base_link" value="-0.10" />
   <xacro:property name="frame_zoff_base_link" value="0.18041" />
-  <xacro:property name="realsense_xoff_frame" value="0.46" />
-  <xacro:property name="realsense_zoff_frame" value="0.06" />
+  <xacro:property name="camera_xoff_frame" value="0.46" />
+  <xacro:property name="camera_zoff_frame" value="0.085" />
   <xacro:property name="velodyne_base_zoff_frame" value="0.326" />
   <xacro:property name="velodyne_xoff_frame" value="${0.245 + 0.02 + 0.0774}" />
@@ -42,5 +42,5 @@
   <link_calibration name="camera_link"
                     parent="mounting_frame_link"
-                    translateX="${realsense_xoff_frame}"
-                    translateZ="${realsense_zoff_frame}" />
+                    translateX="${camera_xoff_frame}"
+                    translateZ="${camera_zoff_frame}" />
 </robot>
